Commit message: Fixed zumo wheels

File: simulation_ws/src/zumo_bot_sims/urdf/robot_training.urdf (robot description, URDF)
Before this commit: robot sumo, 17 links, 16 joints
Links:
- link left_back_link: geometry collision mesh filename=file:///home/takofish/FYP-2022-23/simulation_ws/src/zumo_bo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; visual mesh filename=file:///home/takofish/FYP-2022-23/simulation_ws/src/zumo_bo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
- link left_front_link: geometry collision mesh filename=file:///home/takofish/FYP-2022-23/simulation_ws/src/zumo_bo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; visual mesh filename=file:///home/takofish/FYP-2022-23/simulation_ws/src/zumo_bo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
- link right_back_link: geometry collision mesh filename=file:///home/takofish/FYP-2022-23/simulation_ws/src/zumo_bo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; visual mesh filename=file:///home/takofish/FYP-2022-23/simulation_ws/src/zumo_bo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
- link right_front_link: geometry collision mesh filename=file:///home/takofish/FYP-2022-23/simulation_ws/src/zumo_bo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; visual mesh filename=file:///home/takofish/FYP-2022-23/simulation_ws/src/zumo_bo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

Commit message: Created working lab setup

File: simulation_ws/src/zumo_bot_sims/urdf/robot_training.urdf (robot description, URDF)
Before this commit: robot sumo, 17 links, 16 joints
Links:
- link left_back_link: geometry collision mesh filename=file:///home/csunix/sc20tkkc/FYP-2022-23/simulation_ws/src/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; visual mesh filename=file:///home/csunix/sc20tkkc/FYP-2022-23/simulation_ws/src/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
- link left_front_link: geometry collision mesh filename=file:///home/csunix/sc20tkkc/FYP-2022-23/simulation_ws/src/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; visual mesh filename=file:///home/csunix/sc20tkkc/FYP-2022-23/simulation_ws/src/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
- link right_back_link: geometry collision mesh filename=file:///home/csunix/sc20tkkc/FYP-2022-23/simulation_ws/src/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; visual mesh filename=file:///home/csunix/sc20tkkc/FYP-2022-23/simulation_ws/src/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
- link right_front_link: geometry collision mesh filename=file:///home/csunix/sc20tkkc/FYP-2022-23/simulation_ws/src/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; visual mesh filename=file:///home/csunix/sc20tkkc/FYP-2022-23/simulation_ws/src/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
